File: examples/connector-validation/connector-validation.kicad_pcb (KiCad board)
At the start: 2 copper layers, 355.6 x 213.4 mm, 6 parts

Commit message: Linting fixes.
Routing:
- net /backplane/BA09: track 55.2 -> 52.7 mm
- net /backplane/VCC: track 107.9 -> 105.5 mm
- net /backplane/BA15: track 55.2 -> 52.7 mm
